File: Hardware/BYTE_Sensor_Pack/BYTE_Capacitive/BYTE_Capacitive.sch (KiCad schematic (older format))
At the start: 1 part, among them J1 PCB

Commit message: update capacitive ICs
Parts:
- added C1: 100nF, Capacitor_SMD:C_0603_1608Metric, symbol Device:C_Small
- added C2: 0.1uF, Capacitor_SMD:C_0603_1608Metric, symbol Device:C_Small
- added C3, C4, C5: 1uF, Capacitor_SMD:C_0603_1608Metric, symbol Device:C_Small
- added J?: Conn_01x10, symbol Connector_Generic:Conn_01x10
- added M1: Motor_DC, symbol Motor:Motor_DC
- added R1, R2, R3: 2.2K, Resistor_SMD:R_0603_1608Metric, symbol Device:R_Small
- added U1: AD7147PACPZ-1500R7, BYTE_Sensors:QFN50P400X400X80-25N-D, symbol capacitive_sensor:AD7147PACPZ-1500R7
- added U2: DRV2605YZFR, BYTE_Sensors:BGA9C50P3X3_144X144X62, symbol capacitive_sensor:DRV2605YZFR
Connections:
- new net: M1.1 (+), U2.A3 (OUT+)
- new net: M1.2 (-), U2.C3 (OUT-)
- new net: C1.1, U1.9 (BIAS)
- new net +3V3: C2.1, C3.1, C5.1, R1.1, R2.1, R3.1, U1.11 (VCC), U1.12 (VDRIVE), U2.C2 (VDD)
- new net ACSH: U1.8 (ACSHIELD)
- new net CIN0: U1.19 (CIN0)
- new net CIN1: U1.20 (CIN1)
- new net CIN2: U1.21 (CIN2)
- new net CIN3: U1.22 (CIN3)
- new net EN: U2.A1 (EN)
- new net GND: C1.2, C2.2, C3.2, C4.2, C5.2, U1.10 (GND), U1.14 (ADD0), U1.16 (ADD1), U1.25 (EP), U2.B3 (GND)
- new net GPIO: U1.18 (GPIO)
- new net INT: R3.2, U1.17 (~INT)
- new net IN_TRIG: U2.B1 (IN/TRIG)
- new net REG: C4.1, U2.A2 (REG)
- new net SCL: R1.2, U1.15 (SCLK), U2.C1 (SCL)
- new net SDA: R2.2, U1.13 (SDA), U2.B2 (SDA)
- no-connect marks 0 -> 9
Other:
- moved on the sheet: J1

Commit message: update capacitive sensor board
Parts:
- removed J1: PCB, BYTE_Sensors:Capacitive_PCB, symbol Connector_Generic:Conn_01x06
- removed J?: Conn_01x10, symbol Connector_Generic:Conn_01x10
- removed U2: DRV2605YZFR, BYTE_Sensors:BGA9C50P3X3_144X144X62, symbol capacitive_sensor:DRV2605YZFR
- added J1: input, BYTE_Sensors:Flex_Connector, symbol Connector_Generic:Conn_01x05
- added T1: PCB, BYTE_Sensors:Capacitive_PCB_NoConnector, symbol Connector_Generic:Conn_01x04
- added U2: DRV2605LDGST, BYTE_Sensors:SOP50P490X110-10N, symbol capacitive_sensor:DRV2605LDGST
- C1, C2, C3, C4, C5: footprint Capacitor_SMD:C_0603_1608Metric -> Capacitor_SMD:C_0402_1005Metric
- R1, R2, R3: footprint Resistor_SMD:R_0603_1608Metric -> Resistor_SMD:R_0402_1005Metric
Connections:
- net +3V3: now also J1.5 (Pin_5), U2.10 (VDD), U2.6 (VDD/NC)
- net CIN0: now also T1.4 (Pin_4)
- net CIN1: now also T1.3 (Pin_3)
- net CIN2: now also T1.2 (Pin_2)
- net CIN3: now also T1.1 (Pin_1)
- net EN: now also U2.5 (EN)
- net GND: now also J1.1 (Pin_1), U2.8 (GND)
- net INT: now also J1.4 (Pin_4)
- net IN_TRIG: now also U2.4 (IN/TRIG)
- net REG: now also U2.1 (REG)
- net SCL: now also J1.3 (Pin_3), U2.2 (SCL)
- net SDA: now also J1.2 (Pin_2), U2.3 (SDA)
- net at M1.1 (+): now also U2.9 (OUT-)
- net at M1.2 (-): now also U2.7 (OUT+)
Other:
- moved on the sheet: C4, C5, M1

Commit message: add motor footprint
Parts:
- M1: footprint (none) -> BYTE_Sensors:VLV041235L
Changed lines of the file:
@@
 F 0 "M1" H 10033 1846 50  0000 L CNN
 F 1 "Motor_DC" H 10033 1755 50  0000 L CNN
-F 2 "" H 9875 1760 50  0001 C CNN
+F 2 "BYTE_Sensors:VLV041235L" H 9875 1760 50  0001 C CNN
 F 3 "~" H 9875 1760 50  0001 C CNN
 	1    9875 1850
