File: Hardware/BYTE_Controller_PCB/BYTE_Control_Board.kicad_pcb (KiCad board)
At the start: 2 copper layers, 55 x 19.3 mm, 38 parts, among them J1 8P8C_Shielded, J2 Battery, J3 Expansion, J4 SWD, P1 USB_C_Plug_USB2.0, Q1 DMC2400UV, SW1 GPIO, SW2 GPIO, SW3 RST, U1 MCP73830T-2AAI_MYY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

Commit message: prepare for manufacture
Routing:
- net GND: track 64.7 -> 66.2 mm, vias 17 -> 18
- net /BYTE_SENSOR_2: track 46.8 -> 47.8 mm
Other:
- rule pad_to_mask_clearance: 0.05 -> 0
Changed lines of the file:
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@@
     (thickness 0.8)
     (drawings 25)
-    (tracks 577)
+    (tracks 583)
     (zones 0)
     (modules 38)
@@
     (pad_size 1.05 0.95)
     (pad_drill 0)
-    (pad_to_mask_clearance 0.05)
+    (pad_to_mask_clearance 0)
     (aux_axis_origin 0 0)
     (visible_elements 7FFFFFFF)
     (pcbplotparams
-      (layerselection 0x000c0_7ffffffe)
+      (layerselection 0x010ff_ffffffff)
       (usegerberextensions false)
       (usegerberattributes true)
@@
       (padsonsilk false)
       (subtractmaskfromsilk false)
-      (outputformat 3)
+      (outputformat 1)
       (mirror false)
-      (drillshape 2)
+      (drillshape 0)
       (scaleselection 1)
-      (outputdirectory ""))
+      (outputdirectory "BYTE_Controller_v2.2_Gerbers/"))
   )
   (net 0 "")
@@
       (effects (font (size 1 1) (thickness 0.15)))
     )
+    (fp_circle (center 0 0) (end 0.75 0) (layer F.CrtYd) (width 0.05))
+    (fp_circle (center 0 0) (end 0.5 0) (layer F.Fab) (width 0.1))
     (fp_text user %R (at 0 0) (layer F.Fab)
       (effects (font (size 0.2 0.2) (thickness 0.04)))
     )
-    (fp_circle (center 0 0) (end 0.75 0) (layer F.CrtYd) (width 0.05))
-    (fp_circle (center 0 0) (end 0.5 0) (layer F.Fab) (width 0.1))
     (pad "" smd circle (at 0 0) (size 0.5 0.5) (layers F.Cu F.Mask)
       (solder_mask_margin 0.25) (clearance 0.25))
@@
   (segment (start 160.17 138.45) (end 163.81 138.45) (width 0.2) (layer B.Cu) (net 1))
   (segment (start 159.98 138.26) (end 160.17 138.45) (width 0.2) (layer B.Cu) (net 1))
+  (via (at 158.49 137.13) (size 0.8) (drill 0.4) (layers F.Cu B.Cu) (net 1))
+  (segment (start 158.530004 137.170004) (end 158.49 137.13) (width 0.2) (layer B.Cu) (net 1))
+  (segment (start 159.98 137.170004) (end 158.530004 137.170004) (width 0.2) (layer B.Cu) (net 1))
   (segment (start 160.52 135.82) (end 160.42 135.92) (width 0.25) (layer F.Cu) (net 2))
   (segment (start 160.52 134.44) (end 160.52 135.82) (width 0.25) (layer F.Cu) (net 2))
@@
   (segment (start 144.09 141.19) (end 145.2 140.08) (width 0.2) (layer B.Cu) (net 57))
   (segment (start 152.32 139.31) (end 152.63 139) (width 0.2) (layer B.Cu) (net 57))
-  (segment (start 152.63 139) (end 158.02 139) (width 0.2) (layer B.Cu) (net 57))
   (segment (start 145.2 140.08) (end 152.08 140.08) (width 0.2) (layer B.Cu) (net 57))
   (segment (start 158.02 139) (end 158.54 138.48) (width 0.2) (layer B.Cu) (net 57))
   (segment (start 156.62 139) (end 158.02 139) (width 0.2) (layer F.Cu) (net 57))
   (segment (start 158.02 139) (end 158.54 138.48) (width 0.2) (layer F.Cu) (net 57))
-  (via (at 158.54 138.48) (size 0.8) (drill 0.4) (layers F.Cu B.Cu) (net 57))
+  (via (at 158.54 138.65) (size 0.8) (drill 0.4) (layers F.Cu B.Cu) (net 57))
   (segment (start 138.709996 139.215004) (end 140.165004 139.215004) (width 0.2) (layer B.Cu) (net 57))
   (segment (start 140.165004 139.215004) (end 140.65 139.7) (width 0.2) (layer B.Cu) (net 57))
+  (segment (start 158.19 139) (end 158.54 138.65) (width 0.2) (layer B.Cu) (net 57))
+  (segment (start 152.63 139) (end 157.68 139) (width 0.2) (layer B.Cu) (net 57))
+  (segment (start 157.68 139) (end 158.19 139) (width 0.2) (layer B.Cu) (net 57))
+  (segment (start 157.68 139) (end 158.02 139) (width 0.2) (layer B.Cu) (net 57))
   (via (at 154.879989 126.86092) (size 0.8) (drill 0.4) (layers F.Cu B.Cu) (net 58))
   (segment (start 154.97 126.950931) (end 154.879989 126.86092) (width 0.2) (layer F.Cu) (net 58))
