File: Hardware/BYTE_Sensor_Pack/BYTE_Bite_Base/BYTE_Bite_Base.kicad_pcb (KiCad board)
At the start: 2 copper layers, 12.2 x 9 mm, 1 part, among them J1 Bite

Commit message: prepare for manufacture
Routing:
- removed copper zone on B.Cu, net (none)
Changed lines of the file:
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@@
   (general
     (thickness 1.6)
-    (drawings 4)
+    (drawings 6)
     (tracks 0)
     (zones 0)
@@
     (visible_elements 7FFFFFFF)
     (pcbplotparams
-      (layerselection 0x010fc_ffffffff)
+      (layerselection 0x010ff_ffffffff)
       (usegerberextensions false)
       (usegerberattributes true)
@@
       (outputformat 1)
       (mirror false)
-      (drillshape 1)
+      (drillshape 0)
       (scaleselection 1)
-      (outputdirectory ""))
+      (outputdirectory "BYTE_biteBase_gerber_v1.0"))
   )
   (net 0 "")
@@
     (fp_line (start -5.4 -2.69) (end -5.4 4.31) (layer Edge.Cuts) (width 0.1))
   )
+  (dimension 8.98 (width 0.15) (layer Margin)
+    (gr_text "8.980 mm" (at 147.08 82.67 270) (layer Margin)
+      (effects (font (size 1 1) (thickness 0.15)))
+    )
+    (feature1 (pts (xy 156.59 87.16) (xy 147.793579 87.16)))
+    (feature2 (pts (xy 156.59 78.18) (xy 147.793579 78.18)))
+    (crossbar (pts (xy 148.38 78.18) (xy 148.38 87.16)))
+    (arrow1a (pts (xy 148.38 87.16) (xy 147.793579 86.033496)))
+    (arrow1b (pts (xy 148.38 87.16) (xy 148.966421 86.033496)))
+    (arrow2a (pts (xy 148.38 78.18) (xy 147.793579 79.306504)))
+    (arrow2b (pts (xy 148.38 78.18) (xy 148.966421 79.306504)))
+  )
+  (dimension 12.2 (width 0.15) (layer Margin)
+    (gr_text "12.200 mm" (at 156.72 71.87) (layer Margin)
+      (effects (font (size 1 1) (thickness 0.15)))
+    )
+    (feature1 (pts (xy 162.82 87.18) (xy 162.82 72.583579)))
+    (feature2 (pts (xy 150.62 87.18) (xy 150.62 72.583579)))
+    (crossbar (pts (xy 150.62 73.17) (xy 162.82 73.17)))
+    (arrow1a (pts (xy 162.82 73.17) (xy 161.693496 73.756421)))
+    (arrow1b (pts (xy 162.82 73.17) (xy 161.693496 72.583579)))
+    (arrow2a (pts (xy 150.62 73.17) (xy 151.746504 73.756421)))
+    (arrow2b (pts (xy 150.62 73.17) (xy 151.746504 72.583579)))
+  )
   (gr_circle (center 160.72 84.14) (end 161.11 84.15) (layer F.Mask) (width 2))
   (gr_circle (center 152.97 84.24) (end 153.36 84.25) (layer F.Mask) (width 2))
@@
     (polygon
       (pts
-        (xy 164.2 88.23) (xy 149.05 88.23) (xy 149.05 77.1) (xy 164.2 77.1)
+        (xy 156.49 88.225) (xy 149.05 88.23) (xy 149.05 77.1) (xy 156.49 77.095)
       )
     )
   )
-  (zone (net 0) (net_name "") (layer B.Cu) (hatch edge 0.508)
+  (zone (net 0) (net_name "") (layer F.Cu) (hatch edge 0.508)
     (connect_pads (clearance 0.508))
     (min_thickness 0.254)
@@
     (polygon
       (pts
-        (xy 164.2 88.09) (xy 149.05 88.09) (xy 149.05 76.96) (xy 164.2 76.96)
+        (xy 164.13 88.085) (xy 156.69 88.09) (xy 156.69 76.96) (xy 164.13 76.955)
       )
     )
