File: Hardware/BYTE_Sensor_Pack/BYTE_Flex/Flex_02/Flex_02.kicad_pcb (KiCad board)
At the start: 2 copper layers, 32.5 x 15 mm, 1 part

Commit message: prepare for manufacture
Other:
- rule pad_to_mask_clearance: 0.05 -> 0
- board text added: "Stiffener zone"
Changed lines of the file:
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@@
   (general
     (thickness 0.15)
-    (drawings 24)
+    (drawings 31)
     (tracks 37)
     (zones 0)
@@
     (pad_size 0.2 0.2)
     (pad_drill 0)
-    (pad_to_mask_clearance 0.05)
+    (pad_to_mask_clearance 0)
     (aux_axis_origin 0 0)
     (grid_origin 142.5681 106.14218)
     (visible_elements 7FFFFFFF)
     (pcbplotparams
-      (layerselection 0x010fc_ffffffff)
+      (layerselection 0x014fc_ffffffff)
       (usegerberextensions false)
       (usegerberattributes true)
@@
       (outputformat 1)
       (mirror false)
-      (drillshape 1)
+      (drillshape 0)
       (scaleselection 1)
-      (outputdirectory ""))
+      (outputdirectory "BYTE_Bite_flex_v1.0/"))
   )
   (net 0 "")
@@
       (effects (font (size 0.8 0.8) (thickness 0.12)))
     )
+    (fp_circle (center 0 0) (end -6.75 0) (layer F.SilkS) (width 0.16))
+    (fp_circle (center 0 0) (end -6.55 0) (layer F.Fab) (width 0.1))
     (fp_circle (center 0 0) (end -7 0) (layer F.CrtYd) (width 0.05))
-    (fp_circle (center 0 0) (end -6.55 0) (layer F.Fab) (width 0.1))
-    (fp_circle (center 0 0) (end -6.75 0) (layer F.SilkS) (width 0.16))
     (fp_text user %R (at 0 -8 90) (layer F.Fab)
       (effects (font (size 0.8 0.8) (thickness 0.12)))
@@
     )
   )
+  (dimension 15 (width 0.15) (layer Eco1.User)
+    (gr_text "15.000 mm" (at 130.7381 106.14218 270) (layer Eco1.User)
+      (effects (font (size 1 1) (thickness 0.15)))
+    )
+    (feature1 (pts (xy 142.5981 113.64218) (xy 131.451679 113.64218)))
+    (feature2 (pts (xy 142.5981 98.64218) (xy 131.451679 98.64218)))
+    (crossbar (pts (xy 132.0381 98.64218) (xy 132.0381 113.64218)))
+    (arrow1a (pts (xy 132.0381 113.64218) (xy 131.451679 112.515676)))
+    (arrow1b (pts (xy 132.0381 113.64218) (xy 132.624521 112.515676)))
+    (arrow2a (pts (xy 132.0381 98.64218) (xy 131.451679 99.768684)))
+    (arrow2b (pts (xy 132.0381 98.64218) (xy 132.624521 99.768684)))
+  )
+  (dimension 32.45 (width 0.15) (layer Eco1.User)
+    (gr_text "32.450 mm" (at 151.2931 119.86218) (layer Eco1.User)
+      (effects (font (size 1 1) (thickness 0.15)))
+    )
+    (feature1 (pts (xy 167.5181 106.15218) (xy 167.5181 119.148601)))
+    (feature2 (pts (xy 135.0681 106.15218) (xy 135.0681 119.148601)))
+    (crossbar (pts (xy 135.0681 118.56218) (xy 167.5181 118.56218)))
+    (arrow1a (pts (xy 167.5181 118.56218) (xy 166.391596 119.148601)))
+    (arrow1b (pts (xy 167.5181 118.56218) (xy 166.391596 117.975759)))
+    (arrow2a (pts (xy 135.0681 118.56218) (xy 136.194604 119.148601)))
+    (arrow2b (pts (xy 135.0681 118.56218) (xy 136.194604 117.975759)))
+  )
+  (gr_text "Stiffener zone" (at 170.3181 110.34218) (layer Eco1.User)
+    (effects (font (size 1 1) (thickness 0.15)))
+  )
+  (gr_line (start 167.5181 109.39218) (end 167.5081 102.89218) (layer Eco1.User) (width 0.15))
+  (gr_line (start 164.9681 109.39218) (end 167.5181 109.39218) (layer Eco1.User) (width 0.15))
+  (gr_line (start 164.9681 102.89218) (end 164.9681 109.39218) (layer Eco1.User) (width 0.15))
+  (gr_line (start 167.5081 102.89218) (end 164.9681 102.89218) (layer Eco1.User) (width 0.15))
   (gr_circle (center 159.2281 106.13218) (end 160.9781 106.13218) (layer F.Mask) (width 3.5))
   (gr_poly (pts (xy 159.3981 109.78218) (xy 155.2981 109.78218) (xy 155.2981 102.46218) (xy 159.3981 102.46218)) (layer F.Mask) (width 0.1))
