File: Hardware/BYTE_Sensor_Pack/BYTE_magnetic/BYTE_Magnetic.sch (KiCad schematic (older format))
At the start: 19 parts, among them J1 Input, J2 FSR, M1 Motor_DC, U1 DRV2605LDGS, U2 ADS1115IDGS, U3 PTCA9536BDTMR, U4 SI7210-B-12-IM2, U5 SI7210-B-13-IM2, U6 SI7210-B-14-IM2

Commit message: add manufacturer part number for BOM
Parts:
- C1, C4, C5: manf# (none) -> CL10B105KP8NNNC
- C3, C6, C7: manf# (none) -> CL10B104KA8NNNC
- D1, D2, D3: manf# (none) -> SD0603S040S0R2
- J1, J2: manf# (none) -> -
- M1: manf# (none) -> VLV041235L
- RN1: manf# (none) -> CAY16-221J4LF
- U2: manf# (none) -> ADS1115IDGSR
- U3: manf# (none) -> PTCA9536BDTMR
Changed lines of the file:
@@
 F 2 "BYTE_Sensors:VLV041235L" H 9985 1695 50  0001 C CNN
 F 3 "~" H 9985 1695 50  0001 C CNN
+F 4 "VLV041235L" H 9985 1785 50  0001 C CNN "manf#"
 	1    9985 1785
 	1    0    0    -1
@@
 F 2 "Capacitor_SMD:C_0603_1608Metric" H 9265 2500 50  0001 C CNN
 F 3 "~" H 9265 2500 50  0001 C CNN
+F 4 "CL10B105KP8NNNC" H 9265 2500 50  0001 C CNN "manf#"
 	1    9265 2500
 	1    0    0    -1
@@
 F 2 "Capacitor_SMD:C_0603_1608Metric" H 9135 1120 50  0001 C CNN
 F 3 "~" H 9135 1120 50  0001 C CNN
+F 4 "CL10B105KP8NNNC" H 9135 1120 50  0001 C CNN "manf#"
 	1    9135 1120
 	1    0    0    -1
@@
 F 2 "Capacitor_SMD:C_0603_1608Metric" H 5150 3825 50  0001 C CNN
 F 3 "~" H 5150 3825 50  0001 C CNN
+F 4 "CL10B104KA8NNNC" H 5150 3825 50  0001 C CNN "manf#"
 	1    5150 3825
 	1    0    0    -1
@@
 F 2 "Capacitor_SMD:C_0603_1608Metric" H 7130 3770 50  0001 C CNN
 F 3 "~" H 7130 3770 50  0001 C CNN
+F 4 "CL10B104KA8NNNC" H 7130 3770 50  0001 C CNN "manf#"
 	1    7130 3770
 	1    0    0    -1
@@
 F 2 "Capacitor_SMD:C_0603_1608Metric" H 8955 3825 50  0001 C CNN
 F 3 "~" H 8955 3825 50  0001 C CNN
+F 4 "CL10B104KA8NNNC" H 8955 3825 50  0001 C CNN "manf#"
 	1    8955 3825
 	1    0    0    -1
@@
 F 2 "BYTE_Sensors:Flex_Connector" H 1445 2255 50  0001 C CNN
 F 3 "~" H 1445 2255 50  0001 C CNN
+F 4 "-" H 1445 2255 50  0001 C CNN "manf#"
 	1    1445 2255
 	-1   0    0    1
@@
 F 2 "Package_SO:TSSOP-10_3x3mm_P0.5mm" H 5385 1515 50  0001 C CNN
 F 3 "http://www.ti.com/lit/ds/symlink/ads1113.pdf" H 5335 1115 50  0001 C CNN
+F 4 "ADS1115IDGSR" H 5385 2015 50  0001 C CNN "manf#"
 	1    5385 2015
 	1    0    0    -1
@@
 F 2 "Capacitor_SMD:C_0603_1608Metric" H 5770 1230 50  0001 C CNN
 F 3 "~" H 5770 1230 50  0001 C CNN
+F 4 "CL10B105KP8NNNC" H 5770 1230 50  0001 C CNN "manf#"
 	1    5770 1230
 	1    0    0    -1
@@
 F 2 "" H 3235 2080 50  0001 C CNN
 F 3 "~" H 3235 2080 50  0001 C CNN
+F 4 "-" H 3235 2080 50  0001 C CNN "manf#"
 	1    3235 2080
 	-1   0    0    1
@@
 F 2 "Resistor_SMD:R_Array_Convex_4x0603" V 4425 2600 50  0001 C CNN
 F 3 "~" H 4150 2600 50  0001 C CNN
+F 4 "CAY16-221J4LF" H 4150 2600 50  0001 C CNN "manf#"
 	1    4150 2600
 	-1   0    0    1
@@
 F 2 "Diode_SMD:D_0603_1608Metric" V 5470 4255 50  0001 C CNN
 F 3 "~" V 5470 4255 50  0001 C CNN
+F 4 "SD0603S040S0R2" H 5470 4255 50  0001 C CNN "manf#"
 	1    5470 4255
 	0    1    1    0
@@
 F 2 "Diode_SMD:D_0603_1608Metric" V 7415 4255 50  0001 C CNN
 F 3 "~" V 7415 4255 50  0001 C CNN
+F 4 "SD0603S040S0R2" H 7415 4255 50  0001 C CNN "manf#"
 	1    7415 4255
 	0    1    1    0
@@
 F 2 "Diode_SMD:D_0603_1608Metric" V 9305 4245 50  0001 C CNN
 F 3 "~" V 9305 4245 50  0001 C CNN
+F 4 "SD0603S040S0R2" H 9305 4245 50  0001 C CNN "manf#"
 	1    9305 4245
 	0    1    1    0
@@
 F 2 "BYTE_Sensors:PTCA9416DTMR" H 2300 4755 60  0001 C CNN
 F 3 "https://www.ti.com/lit/ds/symlink/tca9536.pdf?ts=1632417802890&ref_url=https%253A%252F%252Fwww.ti.com%252Fproduct%252FTCA9536" H 2300 5112 60  0001 C CNN
+F 4 "PTCA9536BDTMR" H 1500 4415 50  0001 C CNN "manf#"
 	1    1500 4415
 	1    0    0    -1
